File: KiCAD_PCB/badge.kicad_pcb (KiCad board)
At the start: 2 copper layers, 100 x 100 mm, 156 parts, among them Q1 BC847, Q2 BC847, Q3 BC847, U1 switch, U2 LM1117-3.3, U3 switch, U4 digijoy, U5 switch, U6 wrover, U7 2jumpers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

Commit message: deleted two-transistor helper circuit on gp0/reset that was causing trouble when not connected to an ftdi module same circuit now included in programmer
Parts:
- removed the B1 at (127.1, 82.6)
- removed the B1 at (178.1, 82.6)
- removed Q1 (x2), Q2 (x2): BC847, Package_TO_SOT_SMD:SOT-23
- removed R1 (x2): 10k, LED_SMD:LED_1206_3216Metric_Pad1.42x1.75mm_HandSolder
- removed the U1 at (126.3, 76.4)
- removed the U1 at (177.3, 76.4)
- removed the U3 at (124.0, 96.0)
- removed the U3 at (175.0, 96.0)
- removed the U4 at (114.5, 148.0)
- removed the U4 at (165.5, 148.0)
- removed the U5 at (105.0, 96.0)
- removed the U5 at (156.0, 96.0)
- removed the U6 at (114.9, 143.6)
- removed the U6 at (165.9, 143.6)
- removed the U7 at (111.9, 119.1)
- removed the U7 at (162.9, 119.1)
- removed the U8 at (107.4, 119.1)
- removed the U8 at (158.4, 119.1)
- removed the U9 at (114.5, 120.0)
- removed the U9 at (165.5, 120.0)
- removed the j1 at (98.0, 120.0)
- removed the j1 at (149.0, 120.0)
- added B1: li-ion, badge:powconn, F.Cu at (127.1, 82.6)
- added B1: li-ion, badge:powconn, F.Cu at (178.1, 82.6)
- added D28: mled, LED_SMD:LED_1206_3216Metric_Pad1.42x1.75mm_HandSolder, F.Cu at (108.0, 73.0)
- added REF**: break, badge:break, F.Cu at (140.0, 145.0)
- added REF**: break, badge:break, F.Cu at (140.0, 95.0)
- added U1: switch, badge:switch, F.Cu at (126.3, 76.4)
- added U1: switch, badge:switch, F.Cu at (177.3, 76.4)
- added U3: switch, badge:button, F.Cu at (124.0, 96.0)
- added U3: switch, badge:button, F.Cu at (175.0, 96.0)
- added U4: digijoy, badge:digijoy, F.Cu at (114.5, 148.0)
- added U4: digijoy, badge:digijoy, F.Cu at (165.5, 148.0)
- added U5: switch, badge:button, F.Cu at (105.0, 96.0)
- added U5: switch, badge:button, F.Cu at (156.0, 96.0)
- added U6: wrover, badge:wrover, B.Cu at (114.9, 143.6)
- added U6: wrover, badge:wrover, B.Cu at (165.9, 143.6)
- added U7: 2jumpers, badge:2jumpers, F.Cu at (111.9, 119.1)
- added U7: 2jumpers, badge:2jumpers, F.Cu at (162.9, 119.1)
- added U8: 3jumpers, badge:3jumpers, F.Cu at (107.4, 119.1)
- added U8: 3jumpers, badge:3jumpers, F.Cu at (158.4, 119.1)
- added U9: tft, badge:tft, F.Cu at (114.5, 120.0)
- added j1: ftdi, badge:dcon, F.Cu at (98.0, 120.0)
- added j1: ftdi, badge:dcon, F.Cu at (149.0, 120.0)
- U9: renamed from D28; value mled -> tft; footprint LED_SMD:LED_1206_3216Metric_Pad1.42x1.75mm_HandSolder -> badge:tft
- moved U9 74.3 mm to (165.5, 120.0), turned to 0 degrees
- moved R2 6.99 mm to (131.5, 142.5)
- moved R2 6.99 mm to (182.5, 142.5)
Connections:
- R2 pad 1: Net-(Q2-Pad1) -> Net-(C5-Pad2)
- R2 pad 2: Net-(Q1-Pad2) -> +3V3
- U9 pad 1: (no net) -> GND
- U9 pad 2: (no net) -> Net-(R17-Pad1)
Routing:
- net (no net): track 2519.0 -> 2451.6 mm, vias 101 -> 97
- net Net-(Q1-Pad2): track 52.1 -> 0.00 mm, vias 2 -> 0
- net Net-(Q2-Pad2): track 46.3 -> 0.00 mm
- net Net-(U6-Pad25): track 0.00 -> 42.6 mm, vias 0 -> 1
- net Net-(Q1-Pad3): track 13.1 -> 0.00 mm, vias 1 -> 0
- net +3V3: track 194.5 -> 200.6 mm
- net Net-(Q2-Pad1): track 4.07 -> 0.00 mm
- net Net-(Q1-Pad1): track 2.56 -> 0.00 mm
- net Net-(C5-Pad2): track 96.5 -> 98.7 mm, vias 2 -> 3
- net GND: vias 40 -> 37
